File: KiCAD_EDA/TimeRecordingButton.kicad_sch (KiCad schematic)
At the start: 9 parts, among them J1 USB Micro, J2 Battery, J3 Debug, SW1 SW_Push, U2 PIC16F18114-I/SN

Commit message: KiCAD v2 and removing backup folders.
Parts:
- J2: footprint CustomFootprints:JST_XH_B2B-XH-A_1x02_P2.50mm_SideMount_B -> Connector_JST:JST_PH_B2B-PH-SM4-TB_1x02-1MP_P2.00mm_Vertical
Changed lines of the file:
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@@
       (effects (font (size 1.27 1.27)) (justify right))
     )
-    (property "Footprint" "CustomFootprints:JST_XH_B2B-XH-A_1x02_P2.50mm_SideMount_B" (at 134.62 41.91 0)
+    (property "Footprint" "Connector_JST:JST_PH_B2B-PH-SM4-TB_1x02-1MP_P2.00mm_Vertical" (at 134.62 41.91 0)
       (effects (font (size 1.27 1.27)) hide)
     )
